Commit message: Add a rear caster so the robot stays level
With only a front caster the centre of mass sat over the axle and the body
pitched back about 17 degrees whenever the robot accelerated, tilting the
LiDAR.

File: src/perception_sim/urdf/robot.gazebo.xacro (robot description, xacro)
@@ -5,4 +5,9 @@
   <gazebo reference="right_wheel"><material>Gazebo/Black</material></gazebo>
   <gazebo reference="caster">
+    <material>Gazebo/Black</material>
+    <mu1>0.0</mu1>
+    <mu2>0.0</mu2>
+  </gazebo>
+  <gazebo reference="rear_caster">
     <material>Gazebo/Black</material>
     <mu1>0.0</mu1>

File: src/perception_sim/urdf/robot.urdf.xacro (robot description, xacro)
@@ -66,23 +66,28 @@
   <xacro:wheel prefix="left" y_reflect="1"/>
   <xacro:wheel prefix="right" y_reflect="-1"/>
-  <link name="caster">
-    <visual>
-      <geometry><sphere radius="${wheel_radius/2.0}"/></geometry>
-      <material name="caster"><color rgba="0.1 0.1 0.1 1.0"/></material>
-    </visual>
-    <collision>
-      <geometry><sphere radius="${wheel_radius/2.0}"/></geometry>
-      <surface><friction><ode><mu>0.0</mu><mu2>0.0</mu2></ode></friction></surface>
-    </collision>
-    <inertial>
-      <mass value="0.2"/>
-      <inertia ixx="1e-4" ixy="0" ixz="0" iyy="1e-4" iyz="0" izz="1e-4"/>
-    </inertial>
-  </link>
-  <joint name="caster_joint" type="fixed">
-    <parent link="base_link"/>
-    <child link="caster"/>
-    <origin xyz="${base_length/2.0 - wheel_radius/2.0} 0 ${-base_height/2.0 - wheel_radius/2.0}" rpy="0 0 0"/>
-  </joint>
+  <!-- Casters front and rear so the body cannot pitch when accelerating or braking. -->
+  <xacro:macro name="caster" params="name x_reflect">
+    <link name="${name}">
+      <visual>
+        <geometry><sphere radius="${wheel_radius/2.0}"/></geometry>
+        <material name="caster"><color rgba="0.1 0.1 0.1 1.0"/></material>
+      </visual>
+      <collision>
+        <geometry><sphere radius="${wheel_radius/2.0}"/></geometry>
+        <surface><friction><ode><mu>0.0</mu><mu2>0.0</mu2></ode></friction></surface>
+      </collision>
+      <inertial>
+        <mass value="0.2"/>
+        <inertia ixx="1e-4" ixy="0" ixz="0" iyy="1e-4" iyz="0" izz="1e-4"/>
+      </inertial>
+    </link>
+    <joint name="${name}_joint" type="fixed">
+      <parent link="base_link"/>
+      <child link="${name}"/>
+      <origin xyz="${x_reflect * (base_length/2.0 - wheel_radius/2.0)} 0 ${-base_height/2.0 - wheel_radius/2.0}" rpy="0 0 0"/>
+    </joint>
+  </xacro:macro>
+  <xacro:caster name="caster" x_reflect="1"/>
+  <xacro:caster name="rear_caster" x_reflect="-1"/>
   <!-- Camera at the front of the chassis, looking forward. -->
   <link name="camera_link">

Commit message: Add an IMU and an optional raised payload to the sim robot

File: src/perception_sim/urdf/robot.gazebo.xacro (robot description, xacro)
@@ -4,13 +4,15 @@
   <gazebo reference="left_wheel"><material>Gazebo/Black</material></gazebo>
   <gazebo reference="right_wheel"><material>Gazebo/Black</material></gazebo>
+  <!-- Low but non-zero caster friction: with none at all the robot yaws freely
+       and rolls off a side slope. -->
   <gazebo reference="caster">
     <material>Gazebo/Black</material>
-    <mu1>0.0</mu1>
-    <mu2>0.0</mu2>
+    <mu1>0.1</mu1>
+    <mu2>0.1</mu2>
   </gazebo>
   <gazebo reference="rear_caster">
     <material>Gazebo/Black</material>
-    <mu1>0.0</mu1>
-    <mu2>0.0</mu2>
+    <mu1>0.1</mu1>
+    <mu2>0.1</mu2>
   </gazebo>
   <gazebo reference="camera_link"><material>Gazebo/Red</material></gazebo>
@@ -92,4 +94,40 @@
     </plugin>
   </gazebo>
+  <!-- IMU publishing /imu at 100 Hz in imu_link, physically on the tilted imu_mount.
+       linear_acceleration includes gravity (reads +9.8 on z at rest). -->
+  <xacro:macro name="imu_noise" params="stddev bias">
+    <noise type="gaussian">
+      <mean>0.0</mean>
+      <stddev>${stddev}</stddev>
+      <bias_mean>${bias}</bias_mean>
+      <bias_stddev>${bias / 4.0}</bias_stddev>
+    </noise>
+  </xacro:macro>
+  <gazebo reference="imu_mount">
+    <sensor type="imu" name="imu">
+      <always_on>true</always_on>
+      <update_rate>100.0</update_rate>
+      <imu>
+        <angular_velocity>
+          <x><xacro:imu_noise stddev="0.002" bias="0.0005"/></x>
+          <y><xacro:imu_noise stddev="0.002" bias="0.0005"/></y>
+          <z><xacro:imu_noise stddev="0.002" bias="0.0005"/></z>
+        </angular_velocity>
+        <linear_acceleration>
+          <x><xacro:imu_noise stddev="0.05" bias="0.02"/></x>
+          <y><xacro:imu_noise stddev="0.05" bias="0.02"/></y>
+          <z><xacro:imu_noise stddev="0.05" bias="0.02"/></z>
+        </linear_acceleration>
+      </imu>
+      <plugin name="imu_plugin" filename="libgazebo_ros_imu_sensor.so">
+        <ros>
+          <namespace>/</namespace>
+          <remapping>~/out:=imu</remapping>
+        </ros>
+        <frame_name>imu_link</frame_name>
+        <initial_orientation_as_reference>false</initial_orientation_as_reference>
+      </plugin>
+    </sensor>
+  </gazebo>
   <!-- Forward-facing camera publishing in the optical frame. -->
   <gazebo reference="camera_link">

File: src/perception_sim/urdf/robot.urdf.xacro (robot description, xacro)
@@ -10,4 +10,10 @@
   <xacro:property name="wheel_separation" value="0.34"/>
   <xacro:property name="camera_size" value="0.03"/>
+  <!-- Optional mass on a mast above the LiDAR, like a forklift with its load raised.
+       payload_height is measured from the ground; 0 leaves the robot as it is. -->
+  <xacro:arg name="payload_height" default="0.0"/>
+  <xacro:arg name="payload_mass" default="6.0"/>
+  <xacro:property name="payload_height" value="$(arg payload_height)"/>
+  <xacro:property name="payload_mass" value="$(arg payload_mass)"/>
   <xacro:macro name="box_inertia" params="m x y z">
     <inertial>
@@ -75,5 +81,5 @@
       <collision>
         <geometry><sphere radius="${wheel_radius/2.0}"/></geometry>
-        <surface><friction><ode><mu>0.0</mu><mu2>0.0</mu2></ode></friction></surface>
+        <surface><friction><ode><mu>0.1</mu><mu2>0.1</mu2></ode></friction></surface>
       </collision>
       <inertial>
@@ -133,4 +139,52 @@
     <origin xyz="0 0 ${base_height/2.0 + 0.12}" rpy="0 0 0"/>
   </joint>
+  <!-- IMU at the centre of the chassis. imu_link is where the sensor is meant to be;
+       imu_mount is where it actually sits in simulation, about 1 degree off level, so
+       there is a mounting error for calibrate_imu to find. -->
+  <link name="imu_link"/>
+  <joint name="imu_joint" type="fixed">
+    <parent link="base_link"/>
+    <child link="imu_link"/>
+    <origin xyz="0 0 0" rpy="0 0 0"/>
+  </joint>
+  <link name="imu_mount"/>
+  <joint name="imu_mount_joint" type="fixed">
+    <parent link="base_link"/>
+    <child link="imu_mount"/>
+    <origin xyz="0 0 0" rpy="0.0175 -0.0105 0"/>
+  </joint>
+  <xacro:if value="${payload_height > 0}">
+    <!-- Visual and mass only: no collision, so the LiDAR does not see the mast. -->
+    <xacro:property name="mast_bottom" value="${base_height/2.0 + 0.155}"/>
+    <xacro:property name="mast_top" value="${payload_height - wheel_radius - base_height/2.0 - 0.1}"/>
+    <link name="mast">
+      <visual>
+        <origin xyz="0 0 ${(mast_top - mast_bottom)/2.0}" rpy="0 0 0"/>
+        <geometry><cylinder radius="0.015" length="${mast_top - mast_bottom}"/></geometry>
+        <material name="mast"><color rgba="0.6 0.6 0.6 1.0"/></material>
+      </visual>
+      <inertial>
+        <mass value="0.1"/>
+        <inertia ixx="1e-4" ixy="0" ixz="0" iyy="1e-4" iyz="0" izz="1e-5"/>
+      </inertial>
+    </link>
+    <joint name="mast_joint" type="fixed">
+      <parent link="base_link"/>
+      <child link="mast"/>
+      <origin xyz="0 0 ${mast_bottom}" rpy="0 0 0"/>
+    </joint>
+    <link name="payload">
+      <visual>
+        <geometry><box size="0.2 0.2 0.2"/></geometry>
+        <material name="payload"><color rgba="0.9 0.6 0.1 1.0"/></material>
+      </visual>
+      <xacro:box_inertia m="${payload_mass}" x="0.2" y="0.2" z="0.2"/>
+    </link>
+    <joint name="payload_joint" type="fixed">
+      <parent link="base_link"/>
+      <child link="payload"/>
+      <origin xyz="0 0 ${payload_height - wheel_radius - base_height/2.0}" rpy="0 0 0"/>
+    </joint>
+  </xacro:if>
   <xacro:include filename="$(find perception_sim)/urdf/robot.gazebo.xacro"/>
 </robot>

Commit message: Add a four-wheel skid-steer option to the sim robot

File: src/perception_sim/urdf/robot.gazebo.xacro (robot description, xacro)
@@ -2,6 +2,27 @@
 <robot xmlns:xacro="http://www.ros.org/wiki/xacro">
   <gazebo reference="base_link"><material>Gazebo/Blue</material></gazebo>
-  <gazebo reference="left_wheel"><material>Gazebo/Black</material></gazebo>
-  <gazebo reference="right_wheel"><material>Gazebo/Black</material></gazebo>
+  <xacro:if value="${wheels == 2}">
+    <gazebo reference="left_wheel"><material>Gazebo/Black</material></gazebo>
+    <gazebo reference="right_wheel"><material>Gazebo/Black</material></gazebo>
+  </xacro:if>
+  <xacro:if value="${wheels == 4}">
+    <xacro:macro name="skid_wheel" params="prefix">
+      <!-- Lower sideways friction so the wheels can slide when turning in place, and
+           some contact compliance, like a tyre, to damp skid-steer chatter. -->
+      <gazebo reference="${prefix}_wheel">
+        <material>Gazebo/Black</material>
+        <mu1>1.0</mu1>
+        <mu2>0.6</mu2>
+        <fdir1>1 0 0</fdir1>
+        <kp>200000.0</kp>
+        <kd>2000.0</kd>
+        <minDepth>0.001</minDepth>
+      </gazebo>
+    </xacro:macro>
+    <xacro:skid_wheel prefix="front_left"/>
+    <xacro:skid_wheel prefix="front_right"/>
+    <xacro:skid_wheel prefix="rear_left"/>
+    <xacro:skid_wheel prefix="rear_right"/>
+  </xacro:if>
   <!-- Low but non-zero caster friction: with none at all the robot yaws freely
        and rolls off a side slope. -->
@@ -67,8 +88,21 @@
         <namespace>/</namespace>
       </ros>
-      <left_joint>left_wheel_joint</left_joint>
-      <right_joint>right_wheel_joint</right_joint>
-      <wheel_separation>0.34</wheel_separation>
-      <wheel_diameter>0.12</wheel_diameter>
+      <xacro:if value="${wheels == 2}">
+        <left_joint>left_wheel_joint</left_joint>
+        <right_joint>right_wheel_joint</right_joint>
+        <wheel_separation>0.34</wheel_separation>
+        <wheel_diameter>0.12</wheel_diameter>
+      </xacro:if>
+      <xacro:if value="${wheels == 4}">
+        <num_wheel_pairs>2</num_wheel_pairs>
+        <left_joint>front_left_wheel_joint</left_joint>
+        <right_joint>front_right_wheel_joint</right_joint>
+        <left_joint>rear_left_wheel_joint</left_joint>
+        <right_joint>rear_right_wheel_joint</right_joint>
+        <wheel_separation>0.34</wheel_separation>
+        <wheel_separation>0.34</wheel_separation>
+        <wheel_diameter>0.12</wheel_diameter>
+        <wheel_diameter>0.12</wheel_diameter>
+      </xacro:if>
       <max_wheel_torque>20.0</max_wheel_torque>
       <max_wheel_acceleration>1.0</max_wheel_acceleration>
@@ -90,6 +124,14 @@
       </ros>
       <update_rate>50.0</update_rate>
-      <joint_name>left_wheel_joint</joint_name>
-      <joint_name>right_wheel_joint</joint_name>
+      <xacro:if value="${wheels == 2}">
+        <joint_name>left_wheel_joint</joint_name>
+        <joint_name>right_wheel_joint</joint_name>
+      </xacro:if>
+      <xacro:if value="${wheels == 4}">
+        <joint_name>front_left_wheel_joint</joint_name>
+        <joint_name>front_right_wheel_joint</joint_name>
+        <joint_name>rear_left_wheel_joint</joint_name>
+        <joint_name>rear_right_wheel_joint</joint_name>
+      </xacro:if>
     </plugin>
   </gazebo>

File: src/perception_sim/urdf/robot.urdf.xacro (robot description, xacro)
@@ -14,4 +14,10 @@
   <xacro:arg name="payload_height" default="0.0"/>
   <xacro:arg name="payload_mass" default="6.0"/>
+  <!-- 2: drive wheels in the middle with casters front and rear (default).
+       4: four driven wheels in a rectangle, skid steer; a stance closer to a loader
+       or forklift, used for the tip-over tests on slopes. -->
+  <xacro:arg name="wheels" default="2"/>
+  <xacro:property name="wheels" value="$(arg wheels)"/>
+  <xacro:property name="wheel_base" value="0.28"/>
   <xacro:property name="payload_height" value="$(arg payload_height)"/>
   <xacro:property name="payload_mass" value="$(arg payload_mass)"/>
@@ -50,5 +56,5 @@
     <origin xyz="0 0 ${wheel_radius + base_height/2.0}" rpy="0 0 0"/>
   </joint>
-  <xacro:macro name="wheel" params="prefix y_reflect">
+  <xacro:macro name="wheel" params="prefix y_reflect x:=0.0">
     <link name="${prefix}_wheel">
       <visual>
@@ -66,10 +72,18 @@
       <parent link="base_link"/>
       <child link="${prefix}_wheel"/>
-      <origin xyz="0 ${y_reflect * wheel_separation/2.0} ${-base_height/2.0}" rpy="0 0 0"/>
+      <origin xyz="${x} ${y_reflect * wheel_separation/2.0} ${-base_height/2.0}" rpy="0 0 0"/>
       <axis xyz="0 1 0"/>
     </joint>
   </xacro:macro>
-  <xacro:wheel prefix="left" y_reflect="1"/>
-  <xacro:wheel prefix="right" y_reflect="-1"/>
+  <xacro:if value="${wheels == 2}">
+    <xacro:wheel prefix="left" y_reflect="1"/>
+    <xacro:wheel prefix="right" y_reflect="-1"/>
+  </xacro:if>
+  <xacro:if value="${wheels == 4}">
+    <xacro:wheel prefix="front_left" y_reflect="1" x="${wheel_base/2.0}"/>
+    <xacro:wheel prefix="front_right" y_reflect="-1" x="${wheel_base/2.0}"/>
+    <xacro:wheel prefix="rear_left" y_reflect="1" x="${-wheel_base/2.0}"/>
+    <xacro:wheel prefix="rear_right" y_reflect="-1" x="${-wheel_base/2.0}"/>
+  </xacro:if>
   <!-- Casters front and rear so the body cannot pitch when accelerating or braking. -->
   <xacro:macro name="caster" params="name x_reflect">
@@ -94,6 +108,8 @@
     </joint>
   </xacro:macro>
-  <xacro:caster name="caster" x_reflect="1"/>
-  <xacro:caster name="rear_caster" x_reflect="-1"/>
+  <xacro:if value="${wheels == 2}">
+    <xacro:caster name="caster" x_reflect="1"/>
+    <xacro:caster name="rear_caster" x_reflect="-1"/>
+  </xacro:if>
   <!-- Camera at the front of the chassis, looking forward. -->
   <link name="camera_link">
